File: PCB/Honeydew.kicad_pcb (KiCad board)
At the start: 2 copper layers, 317.8 x 168.8 mm, 326 parts, among them J1 SWD, J2 USB_In, J3 Trackpad, J4 OLED, SW1 MX, SW10 MX, SW11 MX, SW12 MX, SW13 MX, SW14 MX, SW15 MX, SW16 MX, SW17 MX, SW18 MX, SW19 MX, SW2 MX, SW20 MX, SW21 MX, SW22 MX, SW23 MX, SW24 MX, SW25 MX, SW26 MX, SW27 MX, SW28 MX, SW29 MX, SW3 MX, SW30 MX, SW31 MX, SW32 MX, SW33 MX, SW34 MX, SW35 MX, SW36 MX, SW37 MX, SW38 MX, SW39 MX, SW4 MX, SW40 MX, SW41 MX, SW42 MX, SW43 MX, SW44 MX, SW45 MX, SW46 MX, SW47 MX, SW48 MX, SW49 MX, SW5 MX, SW50 MX, SW51 MX, SW52 MX, SW53 MX, SW54 MX, SW55 MX, SW56 MX, SW57 MX, SW58 MX, SW59 MX, SW6 MX, SW60 MX, SW61 MX, SW62 MX, SW63 MX, SW64 Encoder, SW65 Settings, SW66 Reset, SW7 MX, SW8 MX, SW9 MX, U1 AMS1117-3.3, U2 W25Q128JVS, U3 RP2040, U4 PMW3360DM-T2QU, U5 SRV05-4, U6 AP2127K-ADJ, Y1 12MHz

Commit message: Changed RGB LED voltage to 5V.
Parts:
- R5: value NF -> 10k
- moved SW65 6.20 mm to (169.7, 76.9)
- moved SW66 6.20 mm to (169.7, 71.3)
- moved R12 5.40 mm to (167.5, 27.9)
- moved R13 5.34 mm to (172.1, 27.9)
- moved U5 4.85 mm to (169.8, 29.0)
- moved D7 4.42 mm to (58.4, 50.4)
- moved C53 4.42 mm to (112.3, 148.3)
- moved D21 4.42 mm to (120.3, 47.6)
- moved C25 4.42 mm to (175.3, 145.2)
- moved C63 4.42 mm to (200.3, 89.9)
- moved D109 4.42 mm to (218.1, 124.7)
- moved R9 4.42 mm to (171.6, 54.3)
- moved U2 4.42 mm to (179.3, 37.6)
- moved C36 4.42 mm to (59.9, 84.5)
- moved D5 4.42 mm to (20.2, 99.9)
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Connections:
- C23 pad 2: +3V3 -> +5V
- C24 pad 2: +3V3 -> +5V
- C25 pad 2: +3V3 -> +5V
- C26 pad 2: +3V3 -> +5V
- C27 pad 2: +3V3 -> +5V
- C28 pad 2: +3V3 -> +5V
- C29 pad 2: +3V3 -> +5V
- C30 pad 2: +3V3 -> +5V
- C31 pad 2: +3V3 -> +5V
- C32 pad 2: +3V3 -> +5V
- C33 pad 1: +3V3 -> +5V
- C34 pad 2: +3V3 -> +5V
- C35 pad 2: +3V3 -> +5V
- C36 pad 2: +3V3 -> +5V
- C37 pad 2: +3V3 -> +5V
- C38 pad 1: +3V3 -> +5V
- C39 pad 2: +3V3 -> +5V
- C40 pad 2: +3V3 -> +5V
- C41 pad 2: +3V3 -> +5V
- C42 pad 2: +3V3 -> +5V
- C43 pad 1: +3V3 -> +5V
- C44 pad 2: +3V3 -> +5V
- C45 pad 2: +3V3 -> +5V
- C46 pad 2: +3V3 -> +5V
- C47 pad 2: +3V3 -> +5V
- C48 pad 1: +3V3 -> +5V
- C49 pad 2: +3V3 -> +5V
- C50 pad 2: +3V3 -> +5V
- C51 pad 2: +3V3 -> +5V
- C52 pad 2: +3V3 -> +5V
- C53 pad 1: +3V3 -> +5V
- C54 pad 2: +3V3 -> +5V
- C55 pad 2: +3V3 -> +5V
- C56 pad 2: +3V3 -> +5V
- C57 pad 2: +3V3 -> +5V
- C58 pad 2: +3V3 -> +5V
- C59 pad 2: +3V3 -> +5V
- C60 pad 2: +3V3 -> +5V
- C61 pad 2: +3V3 -> +5V
- C62 pad 2: +3V3 -> +5V
- C63 pad 2: +3V3 -> +5V
- C64 pad 2: +3V3 -> +5V
- C65 pad 2: +3V3 -> +5V
- C66 pad 1: +3V3 -> +5V
- C67 pad 2: +3V3 -> +5V
- C68 pad 2: +3V3 -> +5V
- C69 pad 2: +3V3 -> +5V
- C70 pad 2: +3V3 -> +5V
- C71 pad 1: +3V3 -> +5V
- C72 pad 2: +3V3 -> +5V
- C73 pad 2: +3V3 -> +5V
- C74 pad 2: +3V3 -> +5V
- C75 pad 2: +3V3 -> +5V
- C76 pad 1: +3V3 -> +5V
- C77 pad 2: +3V3 -> +5V
- C78 pad 2: +3V3 -> +5V
- C79 pad 2: +3V3 -> +5V
- C80 pad 2: +3V3 -> +5V
- C81 pad 2: +3V3 -> +5V
- C82 pad 2: +3V3 -> +5V
- C83 pad 2: +3V3 -> +5V
- C84 pad 2: +3V3 -> +5V
- C85 pad 2: +3V3 -> +5V
- C86 pad 2: +3V3 -> +5V
- C87 pad 2: +3V3 -> +5V
- C88 pad 2: +3V3 -> +5V
- C89 pad 2: +3V3 -> +5V
- C90 pad 2: +3V3 -> +5V
- C91 pad 2: +3V3 -> +5V
- D100 pad 1: +3V3 -> +5V
- D101 pad 1: +3V3 -> +5V
- D102 pad 1: +3V3 -> +5V
- D103 pad 1: +3V3 -> +5V
- D104 pad 1: +3V3 -> +5V
- D105 pad 1: +3V3 -> +5V
- D106 pad 1: +3V3 -> +5V
- D107 pad 1: +3V3 -> +5V
- D108 pad 1: +3V3 -> +5V
- D109 pad 1: +3V3 -> +5V
- D110 pad 1: +3V3 -> +5V
- D111 pad 1: +3V3 -> +5V
- D112 pad 1: +3V3 -> +5V
- D113 pad 1: +3V3 -> +5V
- D114 pad 1: +3V3 -> +5V
- D115 pad 1: +3V3 -> +5V
- D116 pad 1: +3V3 -> +5V
- D117 pad 1: +3V3 -> +5V
- D118 pad 1: +3V3 -> +5V
- D119 pad 1: +3V3 -> +5V
- D120 pad 1: +3V3 -> +5V
- D121 pad 1: +3V3 -> +5V
- D122 pad 1: +3V3 -> +5V
- D123 pad 1: +3V3 -> +5V
- D124 pad 1: +3V3 -> +5V
- D125 pad 1: +3V3 -> +5V
- D126 pad 1: +3V3 -> +5V
- D127 pad 1: +3V3 -> +5V
- D128 pad 1: +3V3 -> +5V
- D129 pad 1: +3V3 -> +5V
- D130 pad 1: +3V3 -> +5V
- D131 pad 1: +3V3 -> +5V
- D132 pad 1: +3V3 -> +5V
- D133 pad 1: +3V3 -> +5V
- D134 pad 1: +3V3 -> +5V
- D135 pad 1: +3V3 -> +5V
- D67 pad 1: +3V3 -> +5V
- D68 pad 1: +3V3 -> +5V
- D69 pad 1: +3V3 -> +5V
- D70 pad 1: +3V3 -> +5V
- D71 pad 1: +3V3 -> +5V
- D72 pad 1: +3V3 -> +5V
- D73 pad 1: +3V3 -> +5V
- D74 pad 1: +3V3 -> +5V
- D75 pad 1: +3V3 -> +5V
- D76 pad 1: +3V3 -> +5V
- D77 pad 1: +3V3 -> +5V
- D78 pad 1: +3V3 -> +5V
- D79 pad 1: +3V3 -> +5V
- D80 pad 1: +3V3 -> +5V
- D81 pad 1: +3V3 -> +5V
- D82 pad 1: +3V3 -> +5V
- D83 pad 1: +3V3 -> +5V
- D84 pad 1: +3V3 -> +5V
- D85 pad 1: +3V3 -> +5V
- D86 pad 1: +3V3 -> +5V
- D87 pad 1: +3V3 -> +5V
- D88 pad 1: +3V3 -> +5V
- D89 pad 1: +3V3 -> +5V
- D90 pad 1: +3V3 -> +5V
- D91 pad 1: +3V3 -> +5V
- D92 pad 1: +3V3 -> +5V
- D93 pad 1: +3V3 -> +5V
- D94 pad 1: +3V3 -> +5V
- D95 pad 1: +3V3 -> +5V
- D96 pad 1: +3V3 -> +5V
- D97 pad 1: +3V3 -> +5V
- D98 pad 1: +3V3 -> +5V
- D99 pad 1: +3V3 -> +5V
- J1 pad 1: +3V3 -> Net-(J1-Pin_1)
- J1 pad 2: Net-(J1-Pin_2) -> GND
- J1 pad 4: GND -> +3V3
- U3 pad 25: Net-(J1-Pin_2) -> Net-(J1-Pin_1)
Routing:
- net +5V: track 0.00 -> 1679.8 mm, vias 0 -> 44
- net +3V3: track 1899.7 -> 245.7 mm, vias 40 -> 12
- net Net-(J1-Pin_1): track 0.00 -> 15.7 mm
- net Net-(J1-Pin_2): track 12.7 -> 0.00 mm
- net /Comms/VBUS: track 12.6 -> 1.38 mm, vias 2 -> 4
- net Net-(SW66-B): track 25.1 -> 32.4 mm
- net /MCU/Flash: track 36.3 -> 40.1 mm
- net Net-(J2-CC1): track 3.86 -> 6.08 mm
- net Net-(J2-CC2): track 4.06 -> 6.04 mm
- net /Comms/D+: track 21.7 -> 23.0 mm
- net /Comms/D-: track 21.9 -> 23.2 mm
- net Net-(D65-K): track 9.90 -> 10.9 mm
- net GND: track 35.4 -> 35.7 mm, vias 507 -> 488
- added copper zone on F.Cu, net +5V
- added copper zone on F.Cu, net /Comms/VBUS
- removed copper zone on F.Cu, net +3V3
Other:
- board size 317.8 x 168.8 mm -> 317 x 168.8 mm
