File: PCB/Honeydew.kicad_pcb (KiCad board)
At the start: 2 copper layers, 330.1 x 157.7 mm, 364 parts, among them J1 SWD, J2 USB In, J3 Trackpad, J4 OLED, J5 Split_L, J6 Split_R, J7 OLED, J9 RGB_EX, Q1 2N7002, Q5 AO3401A, SW1 CPG151101S11, SW10 CPG151101S11, SW11 CPG151101S11, SW12 CPG151101S11, SW13 CPG151101S11, SW14 CPG151101S11, SW15 CPG151101S11, SW16 CPG151101S11, SW17 CPG151101S11, SW18 CPG151101S11, SW19 CPG151101S11, SW2 CPG151101S11, SW20 CPG151101S11, SW21 CPG151101S11, SW22 CPG151101S11, SW23 CPG151101S11, SW24 CPG151101S11, SW25 CPG151101S11, SW26 CPG151101S11, SW27 CPG151101S11, SW28 CPG151101S11, SW29 CPG151101S11, SW3 CPG151101S11, SW30 CPG151101S11, SW31 CPG151101S11, SW32 CPG151101S11, SW33 CPG151101S11, SW34 CPG151101S11, SW35 CPG151101S11, SW36 CPG151101S11, SW37 CPG151101S11, SW38 CPG151101S11, SW39 CPG151101S11, SW4 CPG151101S11, SW40 CPG151101S11, SW41 CPG151101S11, SW42 CPG151101S11, SW43 CPG151101S11, SW44 CPG151101S11, SW45 CPG151101S11, SW46 CPG151101S11, SW47 CPG151101S11, SW48 CPG151101S11, SW49 CPG151101S11, SW5 CPG151101S11, SW50 CPG151101S11, SW51 CPG151101S11, SW52 CPG151101S11, SW53 CPG151101S11, SW54 CPG151101S11, SW55 CPG151101S11, SW56 CPG151101S11, SW57 CPG151101S11, SW58 CPG151101S11, SW59 CPG151101S11, SW6 CPG151101S11, SW60 CPG151101S11, SW61 CPG151101S11, SW62 CPG151101S11, SW63 CPG151101S11, SW64 Encoder, SW65 Reset, SW66 Reset, SW7 CPG151101S11, SW8 CPG151101S11, SW9 CPG151101S11, U1 AMS1117-3.3, U10 LMV321, U11 TPD4E05U06DQAR, U12 TPD4E05U06DQAR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

Commit message: Added large caps to output of TPS2557. Updated STEP file and file data.
Parts:
- added C104: 47u, Capacitor_SMD:C_1206_3216Metric, B.Cu at (196.5, 84.2)
- added C97: 47u, Capacitor_SMD:C_1206_3216Metric, B.Cu at (192.5, 84.2)
- moved U1 60.7 mm to (197.5, 92.0)
- moved C4 60.4 mm to (196.4, 97.2)
- moved R6 59.0 mm to (225.0, 92.6), turned to 0 degrees
- moved C10 58.7 mm to (203.8, 96.0)
- moved C19 58.4 mm to (205.9, 98.4)
- moved D109 58.3 mm to (264.7, 165.5)
- moved SW38 58.3 mm to (276.1, 134.5)
- moved C46 58.3 mm to (129.8, 132.3)
- moved C1 58.3 mm to (211.1, 132.0)
- moved C22 58.3 mm to (217.3, 156.8)
- moved C27 58.3 mm to (190.5, 160.2)
- moved C41 58.3 mm to (110.3, 131.2)
- moved C80 58.3 mm to (314.2, 148.2)
- moved C90 58.3 mm to (352.9, 145.3)
- moved C93 58.3 mm to (217.0, 162.4)
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Routing:
- net GND: track 39.9 -> 36.3 mm, vias 575 -> 587
- net +3V3: track 183.4 -> 181.4 mm
- net Net-(SW65-B): track 21.2 -> 22.1 mm
- net /Comms - Split/TX: track 118.1 -> 118.7 mm
- net /Comms - Split/RX: track 116.7 -> 117.3 mm
- net Net-(Q5-G): track 1.73 -> 1.17 mm
- net +5VD: track 1718.3 -> 1718.2 mm, vias 104 -> 92
