File: PCB/Expansion.kicad_sch (KiCad schematic)
At the start: 31 parts, among them J3 Trackpad, J4 OLED, J5 OLED_PH, J6 Split_L, J6 Split_R, Q1 AO3401A, U4 PMW3360DM-T2QU, U8 TPD4E05U06DQAR, U9 TPD4E05U06DQAR

Commit message: Additional changes.
Connections:
- net RX: now also U8.2 (IO2), U8.5 (IO4), U8.6 (NC), U8.9 (NC), U9.2 (IO2), U9.5 (IO4), U9.6 (NC), U9.9 (NC); no longer U8.1 (IO1), U8.10 (NC), U8.4 (IO3), U8.7 (NC), U9.1 (IO1), U9.10 (NC), U9.4 (IO3), U9.7 (NC)
- net TX: now also U8.1 (IO1), U8.10 (NC), U8.4 (IO3), U8.7 (NC), U9.1 (IO1), U9.10 (NC), U9.4 (IO3), U9.7 (NC); no longer U8.2 (IO2), U8.5 (IO4), U8.6 (NC), U8.9 (NC), U9.2 (IO2), U9.5 (IO4), U9.6 (NC), U9.9 (NC)
