File: PCB/RGB.kicad_sch (KiCad schematic)
At the start: 69 parts

Commit message: Changed RGB LED voltage to 5V.
Connections:
- net +3V3 renamed +5V
Changed lines of the file:
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@@
     )
+  )
+  (hierarchical_label "+5V" (shape input) (at 275.59 144.78 0) (fields_autoplaced)
+    (effects (font (size 1.27 1.27)) (justify left))
   )
   (hierarchical_label "RGB" (shape input) (at 125.73 33.02 0) (fields_autoplaced)
     (effects (font (size 1.27 1.27)) (justify left))
   )
-  (hierarchical_label "+3V3" (shape input) (at 118.11 22.86 0) (fields_autoplaced)
+  (hierarchical_label "+5V" (shape input) (at 118.11 22.86 0) (fields_autoplaced)
+    (effects (font (size 1.27 1.27)) (justify left))
+  )
+  (hierarchical_label "+5V" (shape input) (at 275.59 63.5 0) (fields_autoplaced)
     (effects (font (size 1.27 1.27)) (justify left))
   )
@@
     (effects (font (size 1.27 1.27)) (justify left))
   )
-  (hierarchical_label "+3V3" (shape input) (at 275.59 104.14 0) (fields_autoplaced)
-    (effects (font (size 1.27 1.27)) (justify left))
-  )
-  (hierarchical_label "+3V3" (shape input) (at 275.59 63.5 0) (fields_autoplaced)
-    (effects (font (size 1.27 1.27)) (justify left))
-  )
   (hierarchical_label "RGB_EX" (shape output) (at 280.67 40.64 180) (fields_autoplaced)
     (effects (font (size 1.27 1.27)) (justify right))
-  )
-  (hierarchical_label "+3V3" (shape input) (at 275.59 144.78 0) (fields_autoplaced)
-    (effects (font (size 1.27 1.27)) (justify left))
   )
   (hierarchical_label "GND" (shape output) (at 275.59 124.46 0) (fields_autoplaced)
     (effects (font (size 1.27 1.27)) (justify left))
   )
-  (hierarchical_label "+3V3" (shape input) (at 118.11 22.86 0) (fields_autoplaced)
+  (hierarchical_label "+5V" (shape input) (at 275.59 104.14 0) (fields_autoplaced)
     (effects (font (size 1.27 1.27)) (justify left))
   )
-  (hierarchical_label "+3V3" (shape input) (at 275.59 63.5 0) (fields_autoplaced)
-    (effects (font (size 1.27 1.27)) (justify left))
-  )

Commit message: Massive mistake corrections and clarifications.
Other:
- moved on the sheet: D100, D101, D102, D103, D104, D105, D106, D107, D108, D109, D110, D111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

Commit message: Rewording of readme. Added files for JLC PCBA. Changed USB C connector and moved it away from board.
Parts:
- D100, D101, D102, D103, D104, D105, D106, D107, D108, D109, D110, D111, D112, D113, D114, D115, D116, D117, D118, D119, D120, D121, D122, D123, D124, D125, D126, D127, D128, D129, D130, D131, D132, D133, D134, D135, D67, D68, D69, D70, D71, D72, D73, D74, D75, D76, D77, D78, D79, D80, D81, D82, D83, D84, D85, D86, D87, D88, D89, D90, D91, D92, D93, D94, D95, D96, D97, D98, D99: LCSC (none) -> C5149201; LCSC part number C5149201 -> (none)

Commit message: Large update.
Parts:
- added J9: RGB_EX, Honeydew:PinHeader_1x04_P2.54mm_Vertical_SIlkless, symbol Connector_Generic:Conn_01x04
- D100, D101, D102, D103, D104, D105, D106, D107, D108, D109, D110, D111, D112, D113, D114, D115, D116, D117, D118, D119, D120, D121, D122, D123, D124, D125, D126, D127, D128, D129, D130, D131, D132, D133, D134, D135, D67, D68, D69, D70, D71, D72, D73, D74, D75, D76, D77, D78, D79, D80, D81, D82, D83, D84, D85, D86, D87, D88, D89, D90, D91, D92, D93, D94, D95, D96, D97, D98, D99: LCSC C5149201 -> C524051
Connections:
- net GND: now also J9.3 (Pin_3), J9.4 (Pin_4)
- net +5V renamed +5VD
- net +5VD: now also J9.2 (Pin_2)
- net RGB_EX: no longer names the net of D131.2 (DOUT)
- net RGB_EX: now also J9.1 (Pin_1)
Other:
- moved on the sheet: D100, D101, D102, D103, D104, D105, D106, D107, D108, D109, D110, D111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
