File: PCB/Comms - SPI.kicad_sch (KiCad schematic)
At the start: 10 parts, among them J3 Trackpad, J4 OLED, J7 OLED, U4 PMW3360DM-T2QU

Commit message: Added large caps to output of TPS2557. Updated STEP file and file data.
Other:
- company: (none) -> Created by Ariamelon (https://github.com/Ariamelon/Honeydew/)
- title: (none) -> Honeydew unified split ergonomic keyboard
Changed lines of the file:
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@@
 (kicad_sch (version 20230121) (generator eeschema)
-  (paper "A5")
+  (paper "A4")
+  (title_block
+    (title "Honeydew unified split ergonomic keyboard")
+    (date "2023-04-08")
+    (rev "V2.0")
+    (company "Created by Ariamelon (https://github.com/Ariamelon/Honeydew/)")
+    (comment 1 "All capacitors 50V unless otherwise specified.")
+    (comment 2 "Licensed under CC BY 4.0.")
+  )
   (junction (at 48.26 16.51) (diameter 0) (color 0 0 0 0)
   )
