File: PCB/Comms - Split.kicad_sch (KiCad schematic)
At the start: 12 parts, among them J1 Split_L, J1 Split_R, U1 TPD4E05U06DQAR

Commit message: Added large caps to output of TPS2557. Updated STEP file and file data.
Other:
- company: (none) -> Created by Ariamelon (https://github.com/Ariamelon/Honeydew/)
- title: (none) -> Honeydew unified split ergonomic keyboard
Changed lines of the file:
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@@
 (kicad_sch (version 20230121) (generator eeschema)
-  (paper "A5")
+  (paper "A4")
+  (title_block
+    (title "Honeydew unified split ergonomic keyboard")
+    (date "2023-04-08")
+    (rev "V2.0")
+    (company "Created by Ariamelon (https://github.com/Ariamelon/Honeydew/)")
+    (comment 1 "All capacitors 50V unless otherwise specified.")
+    (comment 2 "Licensed under CC BY 4.0.")
+  )
   (junction (at 144.78 22.86) (diameter 0) (color 0 0 0 0)
   )

Commit message: Shrunk size of PCB.
Connections:
- net RX: now also U1.2 (IO2), U1.2 (IO2), U1.5 (IO4), U1.5 (IO4), U1.6 (NC), U1.6 (NC), U1.9 (NC), U1.9 (NC); no longer U1.4 (IO3), U1.4 (IO3), U1.7 (NC), U1.7 (NC)
- net TX: now also U1.1 (IO1), U1.1 (IO1), U1.10 (NC), U1.10 (NC), U1.4 (IO3), U1.4 (IO3), U1.7 (NC), U1.7 (NC); no longer U1.2 (IO2), U1.2 (IO2), U1.9 (NC), U1.9 (NC)
