File: PCB/SPI.kicad_sch (KiCad schematic)
At the start: 21 parts, among them J3 Trackpad, J4 OLED_Breakout, J6 SSD1351, U4 PMW3360DM-T2QU

Commit message: BLE version incomplete update.
Parts:
- removed C21 (x4): 1u, Capacitor_SMD:C_0603_1608Metric, symbol Device:C_Small
- removed C38, C43: 100n, Capacitor_SMD:C_0402_1005Metric, symbol Device:C_Small
- removed C39: 10u, Capacitor_SMD:C_0603_1608Metric, symbol Device:C_Small
- removed D57 (x2): 1N4148, Honeydew:D_SOD-323, symbol Device:D_Small
- removed J4: OLED_Breakout, Honeydew:OLED_1.5_SSD1351_128x128, symbol Connector_Generic:Conn_01x07
- removed J6: SSD1351, Honeydew:HRS_FH34SRJ-30S-0.5SH(50), symbol Honeydew:SSD1351
- removed JP1: MISO_Pullup, Jumper:SolderJumper-2_P1.3mm_Open_Pad1.0x1.5mm, symbol Jumper:SolderJumper_2_Open
- removed R29: 51, Resistor_SMD:R_0402_1005Metric, symbol Device:R_Small
- removed R30: 560k, Resistor_SMD:R_0603_1608Metric, symbol Device:R_Small
- added C16: 560p, Capacitor_SMD:C_0402_1005Metric, symbol Device:C_Small
- added C2 (x2): 1u, Capacitor_SMD:C_0603_1608Metric, symbol Device:C_Small
- added FB1 (x2): 600R@100MHz, Inductor_SMD:L_0805_2012Metric, symbol Device:FerriteBead_Small
- added J4: OLED, Honeydew:HRS_FH34SRJ-10S-0.5SH(50), symbol Connector_Generic_MountingPin:Conn_01x10_MountingPin
- added J5: Nice!View, Connector_PinSocket_2.54mm:PinSocket_1x05_P2.54mm_Vertical, symbol Connector_Generic:Conn_01x05
- added JP1: MISO_Pullup, Honeydew:SolderJumper-2_P1.3mm_Open_Pad1.0x1.1mm, symbol Honeydew:SolderJumper_2_Open
- added JP2: VDD_Bridge, Honeydew:SolderJumper-2_P1.3mm_Open_Pad1.0x1.1mm, symbol Honeydew:SolderJumper_2_Open
Connections:
- net +3V3 is gone; now on net VDD: J3.1 (Pin_1), R10.2, R14.2, U4.5 (VDDIO)
- net GND: now also C16.2, C2.2, FB1.2, J4.4 (Pin_4), J4.8 (Pin_8), J4.9 (Pin_9), J4.MP (MountPin), J5.2 (Pin_2)
- net MISO: now also JP1.1 (A)
- net MOSI: now also J4.2 (Pin_2), J5.5 (Pin_5)
- net OLED_CS: now also J4.3 (Pin_3), J5.1 (Pin_1)
- net SCK: now also J4.1 (Pin_1), J5.4 (Pin_4)
- net at R14.1: now also JP1.2 (B)
- net +2V renamed VDD
- net VDD: now also J5.3 (Pin_3), JP2.2 (B)
- new net VDDA: C2.1, FB1.1, J4.6 (Pin_6)
- new net VDDF: C16.1, C2.1, FB1.2, J4.5 (Pin_5), J4.7 (Pin_7), JP2.1 (A)
- new net VSSA: C2.2, FB1.1, J4.10 (Pin_10)
- no-connect marks 11 -> 5
Other:
- note added: "Solder jumper if Nice!View isn't used"
- moved on the sheet: R14
