File: PCB/SPI.kicad_sch (KiCad schematic)
At the start: 21 parts, among them J3 Trackpad, J4 OLED_Breakout, J6 SSD1351, U4 PMW3360DM-T2QU

Commit message: 28/07/2023 update
Removed center ring encoder, cirque trackpad and PMW3360 support. Added VIK header and hole in the center of the PCB for the Kiwano. Changed JST connectors back to 20 pin FFC. Total rearrangement of parts in keyboard center. Stitched ground planes together. Added USB module to board rather than have it be separate.
Parts:
- removed C21 (x4): 1u, Capacitor_SMD:C_0603_1608Metric, symbol Device:C_Small
- removed C26: 4u7, Capacitor_SMD:C_0603_1608Metric, symbol Device:C_Small
- removed C27, C38, C43: 100n, Capacitor_SMD:C_0402_1005Metric, symbol Device:C_Small
- removed C39: 10u, Capacitor_SMD:C_0603_1608Metric, symbol Device:C_Small
- removed D57 (x2): 1N4148, Honeydew:D_SOD-323, symbol Device:D_Small
- removed J3: Trackpad, Honeydew:HRS_FH34SRJ-12S-0.5SH(50), symbol Connector_Generic_MountingPin:Conn_01x12_MountingPin
- removed J4: OLED_Breakout, Honeydew:OLED_1.5_SSD1351_128x128, symbol Connector_Generic:Conn_01x07
- removed J6: SSD1351, Honeydew:HRS_FH34SRJ-30S-0.5SH(50), symbol Honeydew:SSD1351
- removed JP2: MISO Pullup, Honeydew:SolderJumper-2_P1.2mm_Open_Pad1.0x1.0mm, symbol Honeydew:SolderJumper_2_Open
- removed R10, R14: 10k, Resistor_SMD:R_0402_1005Metric, symbol Device:R_Small
- removed R11: 39, Resistor_SMD:R_0402_1005Metric, symbol Device:R_Small
- removed R29: 51, Resistor_SMD:R_0402_1005Metric, symbol Device:R_Small
- removed R30: 560k, Resistor_SMD:R_0603_1608Metric, symbol Device:R_Small
- removed U4: PMW3360DM-T2QU, Honeydew:IC_PMW3360DM-T2QU, symbol Ogen:PMW3360DM-T2QU
Connections:
- no-connect marks 11 -> 0
