File: PCB/Plate.kicad_pcb (KiCad board)
At the start: 2 copper layers, 317 x 171.1 mm, 63 parts, among them SW1 MX, SW10 MX, SW11 MX, SW12 MX, SW13 MX, SW14 MX, SW15 MX, SW16 MX, SW17 MX, SW18 MX, SW19 MX, SW2 MX, SW20 MX, SW21 MX, SW22 MX, SW23 MX, SW24 MX, SW25 MX, SW26 MX, SW27 MX, SW28 MX, SW29 MX, SW3 MX, SW30 MX, SW4 MX, SW5 MX, SW6 MX, SW61 MX, SW62 MX, SW7 MX, SW8 MX, SW9 MX

Commit message: Added PH2.0 header for OLED. Changed plate to accommodate headers.
Parts:
- removed the SW61 at (153.7, 170.1)
- removed SW62: MX, Honeydew:Cutout_MX_Tight
- added SW61: MX, Honeydew:Cutout_MX_Tight, F.Cu at (176.9, 191.9)
- added SW61: MX, Honeydew:Cutout_MX_Tight, B.Cu at (155.5, 189.1)
- moved SW10 19.1 mm to (302.3, 133.6)
- moved SW10 19.1 mm to (51.5, 133.6)
- moved SW13 19.1 mm to (84.1, 99.9)
- moved SW15 19.1 mm to (282.8, 135.7)
- moved SW15 19.1 mm to (71.0, 135.7)
- moved SW22 19.1 mm to (227.5, 95.0)
- moved SW22 19.1 mm to (126.4, 95.0)
- moved SW24 19.1 mm to (240.5, 130.8)
- moved SW24 19.1 mm to (113.4, 130.8)
- moved SW5 19.1 mm to (321.1, 129.3)
- moved SW5 19.1 mm to (32.8, 129.3)
- moved SW8 19.1 mm to (64.5, 97.8)
- moved SW13 19.1 mm to (269.8, 99.9)
- moved SW8 19.1 mm to (289.3, 97.8)
- moved SW12 19.1 mm to (263.3, 82.0)
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Other:
- outline, holes or cut-outs redrawn

Commit message: More V1.1 updates
Parts:
- SW1 (x2), SW10 (x2), SW11 (x2), SW12 (x2), SW13 (x2), SW14 (x2), SW15 (x2), SW16 (x2), SW17 (x2), SW18 (x2), SW19 (x2), SW2 (x2), SW20 (x2), SW21 (x2), SW22 (x2), SW23 (x2), SW24 (x2), SW25 (x2), SW26 (x2), SW27 (x2), SW28 (x2), SW29 (x2), SW3 (x2), SW30 (x2), SW4 (x2), SW5 (x2), SW6 (x2), SW61 (x3), SW7 (x2), SW8 (x2), SW9 (x2): footprint Honeydew:Cutout_MX_Tight -> Honeydew:MX100
- moved SW29 0.60 mm to (223.8, 140.9)
- moved SW30 0.60 mm to (135.0, 176.6)
- moved SW20 0.60 mm to (99.3, 151.6)
- moved SW20 0.60 mm to (254.7, 151.6)
- moved SW29 0.60 mm to (130.2, 140.9)
- moved SW30 0.60 mm to (219.0, 176.6)
- moved SW18 0.60 mm to (250.6, 103.2)
- moved SW14 0.60 mm to (77.6, 118.4)
- moved SW19 0.60 mm to (96.9, 121.1)
- moved SW2 0.60 mm to (52.4, 76.2)
- moved SW9 0.60 mm to (58.1, 116.3)
- moved SW14 0.60 mm to (276.4, 118.4)
- moved SW18 0.60 mm to (103.4, 103.2)
- moved SW19 0.60 mm to (257.1, 121.1)
- moved SW2 0.60 mm to (301.6, 76.2)
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Other:
- board size 317 x 171.1 mm -> 316.7 x 174.4 mm

Commit message: Moved position of USB-C ports further out.
Parts:
- removed the SW1 at (295.1, 58.3)
- removed the SW1 at (58.9, 58.3)
- removed the SW10 at (302.4, 134.2)
- removed the SW10 at (51.6, 134.2)
- removed the SW11 at (256.8, 64.7)
- removed the SW11 at (97.2, 64.7)
- removed the SW12 at (263.3, 82.6)
- removed the SW12 at (90.7, 82.6)
- removed the SW13 at (269.9, 100.5)
- removed the SW13 at (84.1, 100.5)
- removed the SW14 at (276.4, 118.4)
- removed the SW14 at (77.6, 118.4)
- removed the SW15 at (282.9, 136.3)
- removed the SW15 at (71.1, 136.3)
- removed the SW16 at (237.6, 67.4)
- removed the SW16 at (116.4, 67.4)
- removed the SW17 at (244.1, 85.3)
- removed the SW17 at (109.9, 85.3)
- removed the SW18 at (250.6, 103.2)
- removed the SW18 at (103.4, 103.2)
- removed the SW19 at (257.1, 121.1)
- removed the SW19 at (96.9, 121.1)
- removed the SW2 at (301.6, 76.2)
- removed the SW2 at (52.4, 76.2)
- removed the SW20 at (254.7, 151.6)
- removed the SW20 at (99.3, 151.6)
- removed the SW21 at (221.0, 77.7)
- removed the SW21 at (133.0, 77.7)
- removed the SW22 at (227.5, 95.6)
- removed the SW22 at (126.5, 95.6)
- removed the SW23 at (234.1, 113.5)
- removed the SW23 at (119.9, 113.5)
- removed the SW24 at (240.6, 131.4)
- removed the SW24 at (113.4, 131.4)
- removed the SW25 at (235.1, 161.7)
- removed the SW25 at (118.9, 161.7)
- removed the SW26 at (204.2, 87.2)
- removed the SW26 at (149.8, 87.2)
- removed the SW27 at (210.7, 105.1)
- removed the SW27 at (143.3, 105.1)
- removed the SW28 at (217.2, 123.0)
- removed the SW28 at (136.8, 123.0)
- removed the SW29 at (223.8, 140.9)
- removed the SW29 at (130.2, 140.9)
- removed the SW3 at (308.1, 94.1)
- removed the SW3 at (45.9, 94.1)
- removed the SW30 at (219.0, 176.6)
- removed the SW30 at (135.0, 176.6)
- removed the SW4 at (314.6, 112.0)
- removed the SW4 at (39.4, 112.0)
- removed the SW5 at (321.1, 129.9)
- removed the SW5 at (32.9, 129.9)
- removed the SW6 at (276.4, 62.6)
- removed the SW6 at (77.6, 62.6)
- removed the SW61 at (177.0, 192.5)
- removed the SW61 at (198.4, 189.7)
- removed the SW61 at (155.6, 189.7)
- removed the SW7 at (282.9, 80.5)
- removed the SW7 at (71.1, 80.5)
- removed the SW8 at (289.4, 98.4)
- removed the SW8 at (64.6, 98.4)
- removed the SW9 at (295.9, 116.3)
- removed the SW9 at (58.1, 116.3)
- added SW1: CPG151101S11, Honeydew:MX100, F.Cu at (46.8, 49.9)
- added SW10: CPG151101S11, Honeydew:MX100, F.Cu at (46.1, 126.2)
- added SW11: CPG151101S11, Honeydew:MX100, F.Cu at (85.5, 52.9)
- added SW12: CPG151101S11, Honeydew:MX100, F.Cu at (80.6, 71.3)
- added SW13: CPG151101S11, Honeydew:MX100, F.Cu at (75.6, 89.7)
- added SW14: CPG151101S11, Honeydew:MX100, F.Cu at (70.7, 108.1)
- added SW15: CPG151101S11, Honeydew:MX100, F.Cu at (65.8, 126.5)
- added SW16: CPG151101S11, Honeydew:MX100, F.Cu at (104.9, 54.0)
- added SW17: CPG151101S11, Honeydew:MX100, F.Cu at (100.0, 72.4)
- added SW18: CPG151101S11, Honeydew:MX100, F.Cu at (95.1, 90.8)
- added SW19: CPG151101S11, Honeydew:MX100, F.Cu at (90.1, 109.2)
- added SW2: CPG151101S11, Honeydew:MX100, F.Cu at (41.9, 68.3)
- added SW20: CPG151101S11, Honeydew:MX100, F.Cu at (95.2, 139.3)
- added SW21: CPG151101S11, Honeydew:MX100, F.Cu at (122.3, 62.7)
- added SW22: CPG151101S11, Honeydew:MX100, F.Cu at (117.4, 81.1)
- added SW23: CPG151101S11, Honeydew:MX100, F.Cu at (112.4, 99.5)
- added SW24: CPG151101S11, Honeydew:MX100, F.Cu at (107.5, 117.9)
- added SW25: CPG151101S11, Honeydew:MX100, F.Cu at (115.6, 147.7)
- added SW26: CPG151101S11, Honeydew:MX100, F.Cu at (139.9, 70.7)
- added SW27: CPG151101S11, Honeydew:MX100, F.Cu at (134.9, 89.1)
- added SW28: CPG151101S11, Honeydew:MX100, F.Cu at (130.0, 107.5)
- added SW29: CPG151101S11, Honeydew:MX100, F.Cu at (125.1, 125.9)
- added SW3: CPG151101S11, Honeydew:MX100, F.Cu at (37.0, 86.7)
- added SW30: CPG151101S11, Honeydew:MX100, F.Cu at (132.9, 161.1)
- added SW31: CPG151101S11, Honeydew:MX100, F.Cu at (210.1, 70.7)
- added SW32: CPG151101S11, Honeydew:MX100, F.Cu at (215.1, 89.1)
- added SW33: CPG151101S11, Honeydew:MX100, F.Cu at (220.0, 107.5)
- added SW34: CPG151101S11, Honeydew:MX100, F.Cu at (224.9, 125.9)
- added SW35: CPG151101S11, Honeydew:MX100, F.Cu at (217.1, 161.1)
- added SW36: CPG151101S11, Honeydew:MX100, F.Cu at (227.7, 62.7)
- added SW37: CPG151101S11, Honeydew:MX100, F.Cu at (232.6, 81.1)
- added SW38: CPG151101S11, Honeydew:MX100, F.Cu at (237.6, 99.5)
- added SW39: CPG151101S11, Honeydew:MX100, F.Cu at (242.5, 117.9)
- added SW4: CPG151101S11, Honeydew:MX100, F.Cu at (32.0, 105.1)
- added SW40: CPG151101S11, Honeydew:MX100, F.Cu at (234.4, 147.7)
- added SW41: CPG151101S11, Honeydew:MX100, F.Cu at (245.1, 54.0)
- added SW42: CPG151101S11, Honeydew:MX100, F.Cu at (250.0, 72.4)
- added SW43: CPG151101S11, Honeydew:MX100, F.Cu at (254.9, 90.8)
- added SW44: CPG151101S11, Honeydew:MX100, F.Cu at (259.9, 109.2)
- added SW45: CPG151101S11, Honeydew:MX100, F.Cu at (254.8, 139.3)
- added SW46: CPG151101S11, Honeydew:MX100, F.Cu at (264.5, 52.9)
- added SW47: CPG151101S11, Honeydew:MX100, F.Cu at (269.4, 71.3)
- added SW48: CPG151101S11, Honeydew:MX100, F.Cu at (274.4, 89.7)
- added SW49: CPG151101S11, Honeydew:MX100, F.Cu at (279.3, 108.1)
- added SW5: CPG151101S11, Honeydew:MX100, F.Cu at (27.1, 123.5)
- added SW50: CPG151101S11, Honeydew:MX100, F.Cu at (284.2, 126.5)
- added SW51: CPG151101S11, Honeydew:MX100, F.Cu at (284.1, 52.5)
- added SW52: CPG151101S11, Honeydew:MX100, F.Cu at (289.1, 70.9)
- added SW53: CPG151101S11, Honeydew:MX100, F.Cu at (294.0, 89.4)
- added SW54: CPG151101S11, Honeydew:MX100, F.Cu at (298.9, 107.8)
- added SW55: CPG151101S11, Honeydew:MX100, F.Cu at (303.9, 126.2)
- added SW56: CPG151101S11, Honeydew:MX100, F.Cu at (303.2, 49.9)
- added SW57: CPG151101S11, Honeydew:MX100, F.Cu at (308.1, 68.3)
- added SW58: CPG151101S11, Honeydew:MX100, F.Cu at (313.0, 86.7)
- added SW59: CPG151101S11, Honeydew:MX100, F.Cu at (318.0, 105.1)
- added SW6: CPG151101S11, Honeydew:MX100, F.Cu at (65.9, 52.5)
- added SW60: CPG151101S11, Honeydew:MX100, F.Cu at (322.9, 123.5)
- added SW61: CPG151101S11, Honeydew:MX100, F.Cu at (153.6, 173.1)
- added SW62: CPG151101S11, Honeydew:MX100, F.Cu at (175.0, 175.9)
- added SW63: CPG151101S11, Honeydew:MX100, F.Cu at (196.4, 173.1)
- added SW7: CPG151101S11, Honeydew:MX100, F.Cu at (60.9, 70.9)
- added SW8: CPG151101S11, Honeydew:MX100, F.Cu at (56.0, 89.4)
- added SW9: CPG151101S11, Honeydew:MX100, F.Cu at (51.1, 107.8)
Other:
- board size 316.7 x 174.4 mm -> 323.3 x 165 mm

Commit message: Shrunk size of PCB.
Parts:
- SW1, SW10, SW11, SW12, SW13, SW14, SW15, SW16, SW17, SW18, SW19, SW2, SW20, SW21, SW22, SW23, SW24, SW25, SW26, SW27, SW28, SW29, SW3, SW30, SW31, SW32, SW33, SW34, SW35, SW36, SW37, SW38, SW39, SW4, SW40, SW41, SW42, SW43, SW44, SW45, SW46, SW47, SW48, SW49, SW5, SW50, SW51, SW52, SW53, SW54, SW55, SW56, SW57, SW58, SW59, SW6, SW60, SW61, SW62, SW63, SW7, SW8, SW9: moved to B.Cu
- moved SW37 48.8 mm to (271.1, 111.1), turned to -165 degrees
- moved SW44 48.8 mm to (298.4, 139.2), turned to -165 degrees
- moved SW46 48.8 mm to (303.0, 82.9), turned to -165 degrees
- moved SW54 48.8 mm to (337.4, 137.8), turned to -165 degrees
- moved SW33 48.8 mm to (258.5, 137.5), turned to -165 degrees
- moved SW49 48.8 mm to (317.8, 138.1), turned to -165 degrees
- moved SW57 48.8 mm to (346.6, 98.3), turned to -165 degrees
- moved SW59 48.8 mm to (356.5, 135.1), turned to -165 degrees
- moved SW43 48.8 mm to (293.4, 120.8), turned to -165 degrees
- moved SW32 48.8 mm to (253.6, 119.1), turned to -165 degrees
- moved SW53 48.8 mm to (332.5, 119.4), turned to -165 degrees
- moved SW41 48.8 mm to (283.6, 84.0), turned to -165 degrees
- moved SW35 48.8 mm to (255.6, 191.1), turned to -135 degrees
- moved SW45 48.8 mm to (293.3, 169.3), turned to -165 degrees
- moved SW38 48.8 mm to (276.1, 129.5), turned to -165 degrees
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Other:
- board size 323.3 x 165 mm -> 325.2 x 147.9 mm
- board text added: "Encoder"
- board text added: "SW50"

Commit message: Added plate DXF and gerbers. Removed split comms ports and ideal diode.
Other:
- board size 325.2 x 147.9 mm -> 332.7 x 160 mm
- board text removed: "Encoder"
- board text removed: "SW50"

Commit message: 17/04/2023 large update.
Parts:
- removed the SW27 at (166.4, 119.1)
- removed SW28, SW56: CPG151101S11, Honeydew:MX100
- removed the SW51 at (322.6, 82.5)
- added H4: M3, Honeydew:MountingHole_3.2mm_M3_Pad, F.Cu at (244.4, 84.6)
- added H5: M3, Honeydew:MountingHole_3.2mm_M3_Pad, F.Cu at (175.6, 84.6)
- added H6: M3, Honeydew:MountingHole_3.2mm_M3_Pad, F.Cu at (88.5, 179.6)
- added H7: M3, Honeydew:MountingHole_3.2mm_M3_Pad, F.Cu at (331.5, 179.6)
- added H8: M3, Honeydew:MountingHole_3.2mm_M3_Pad, F.Cu at (250.0, 217.5)
- added H9: M3, Honeydew:MountingHole_3.2mm_M3_Pad, F.Cu at (169.7, 217.5)
- added SW27: CPG151101S11, Honeydew:MX100, B.Cu at (166.4, 131.7)
- added SW27: CPG151101S11, Honeydew:MX100, B.Cu at (161.5, 150.1)
- added SW51: CPG151101S11, Honeydew:MX100, B.Cu at (322.6, 95.1)
- added SW51: CPG151101S11, Honeydew:MX100, B.Cu at (341.7, 92.5)
- added SWr: CPG151101S11, Honeydew:MX200, B.Cu at (210.0, 222.1)
- moved SW60 12.6 mm to (361.4, 166.1)
- moved SW47 12.6 mm to (307.9, 113.8)
- moved SW46 12.6 mm to (303.0, 95.4)
- moved SW10 12.6 mm to (77.6, 168.7)
- moved SW39 12.6 mm to (281.0, 160.5)
- moved SW1 12.6 mm to (78.3, 92.5)
- moved SW17 12.6 mm to (131.5, 114.9)
- moved SW16 12.6 mm to (136.4, 96.5)
- moved SW43 12.6 mm to (293.4, 133.3)
- moved SW2 12.6 mm to (73.4, 110.9)
- moved SW58 12.6 mm to (351.5, 129.3)
- moved SW52 12.6 mm to (327.6, 113.5)
- moved SW55 12.6 mm to (342.4, 168.7)
- moved SW20 12.6 mm to (126.7, 181.9)
- moved SW32 12.6 mm to (253.6, 131.7)
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Other:
- board size 332.7 x 160 mm -> 325.2 x 151 mm

Commit message: Rerouting.
Parts:
- turned SWr to 180 degrees
Other:
- outline, holes or cut-outs redrawn
Changed lines of the file:
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@@
   )
   (footprint "Honeydew:MX200" (layer "B.Cu")
-    (at 209.999996 222.050004)
+    (at 209.999996 222.050004 180)
     (property "Description" "Kailh hotswap sockets")
     (property "LCSC" "C5184526")
@@
     (fp_line (start 19.05 9.525) (end 19.05 -9.525)
       (stroke (width 0.12) (type solid)) (layer "Dwgs.User"))
-    (fp_line (start -15.40625 5.5) (end -15.40625 -7.500008)
-      (stroke (width 0.12) (type default)) (layer "Edge.Cuts"))
-    (fp_line (start -14.90625 -8.000008) (end -8.90625 -8.000008)
-      (stroke (width 0.12) (type default)) (layer "Edge.Cuts"))
-    (fp_line (start -8.90625 6) (end -14.90625 6)
-      (stroke (width 0.12) (type default)) (layer "Edge.Cuts"))
-    (fp_line (start -8.40625 -7.500008) (end -8.40625 5.5)
-      (stroke (width 0.12) (type default)) (layer "Edge.Cuts"))
-    (fp_line (start -7 6.5) (end -7 -6.5)
-      (stroke (width 0.12) (type default)) (layer "Edge.Cuts"))
-    (fp_line (start -6.5 -7) (end 6.499672 -7.000007)
-      (stroke (width 0.12) (type default)) (layer "Edge.Cuts"))
-    (fp_line (start 6.5 7) (end -6.5 7)
-      (stroke (width 0.12) (type default)) (layer "Edge.Cuts"))
-    (fp_line (start 6.999672 -6.500007) (end 7 6.5)
-      (stroke (width 0.12) (type default)) (layer "Edge.Cuts"))
-    (fp_line (start 8.40625 -7.500008) (end 8.40625 5.5)
-      (stroke (width 0.12) (type default)) (layer "Edge.Cuts"))
-    (fp_line (start 8.90625 6) (end 14.90625 6)
-      (stroke (width 0.12) (type default)) (layer "Edge.Cuts"))
-    (fp_line (start 14.90625 -8.000008) (end 8.90625 -8.000008)
-      (stroke (width 0.12) (type default)) (layer "Edge.Cuts"))
-    (fp_line (start 15.40625 5.5) (end 15.40625 -7.500008)
-      (stroke (width 0.12) (type default)) (layer "Edge.Cuts"))
-    (fp_arc (start -15.40625 -7.500008) (mid -15.259803 -7.853561) (end -14.90625 -8.000008)
+    (fp_line (start -15.313 5.5) (end -15.313 -7.5)
+      (stroke (width 0.1) (type default)) (layer "Edge.Cuts"))
+    (fp_line (start -14.813 -8) (end -9.063 -8)
+      (stroke (width 0.1) (type default)) (layer "Edge.Cuts"))
+    (fp_line (start -9.063 6) (end -14.813 6)
+      (stroke (width 0.1) (type default)) (layer "Edge.Cuts"))
+    (fp_line (start -8.563 -7.5) (end -8.563 5.5)
+      (stroke (width 0.1) (type default)) (layer "Edge.Cuts"))
+    (fp_line (start -7 -6.5) (end -7 6.5)
+      (stroke (width 0.1) (type default)) (layer "Edge.Cuts"))
+    (fp_line (start -6.5 7) (end 6.5 7)
+      (stroke (width 0.1) (type default)) (layer "Edge.Cuts"))
+    (fp_line (start 6.5 -7) (end -6.5 -7)
+      (stroke (width 0.1) (type default)) (layer "Edge.Cuts"))
+    (fp_line (start 7 6.5) (end 7 -6.5)
+      (stroke (width 0.1) (type default)) (layer "Edge.Cuts"))
+    (fp_line (start 8.563 5.5) (end 8.563 -7.5)
+      (stroke (width 0.1) (type default)) (layer "Edge.Cuts"))
+    (fp_line (start 9.063 -8) (end 14.813 -8)
+      (stroke (width 0.1) (type default)) (layer "Edge.Cuts"))
+    (fp_line (start 14.813 6) (end 9.063 6)
+      (stroke (width 0.1) (type default)) (layer "Edge.Cuts"))
+    (fp_line (start 15.313 -7.5) (end 15.313 5.5)
+      (stroke (width 0.1) (type default)) (layer "Edge.Cuts"))
+    (fp_arc (start -15.313 -7.5) (mid -15.166581 -7.853581) (end -14.813 -8)
       (stroke (width 0.1) (type solid)) (layer "Edge.Cuts"))
-    (fp_arc (start -14.90625 6) (mid -15.259803 5.853553) (end -15.40625 5.5)
+    (fp_arc (start -14.813 6) (mid -15.166562 5.853562) (end -15.313 5.5)
       (stroke (width 0.1) (type solid)) (layer "Edge.Cuts"))
-    (fp_arc (start -8.90625 -8.000008) (mid -8.552697 -7.853561) (end -8.40625 -7.500008)
+    (fp_arc (start -9.063 -8) (mid -8.70946 -7.85354) (end -8.563 -7.5)
       (stroke (width 0.1) (type solid)) (layer "Edge.Cuts"))
-    (fp_arc (start -8.40625 5.5) (mid -8.552697 5.853553) (end -8.90625 6)
+    (fp_arc (start -8.563 5.5) (mid -8.709451 5.853549) (end -9.063 6)
       (stroke (width 0.1) (type solid)) (layer "Edge.Cuts"))
     (fp_arc (start -7 -6.5) (mid -6.853553 -6.853553) (end -6.5 -7)
@@
     (fp_arc (start -6.5 7) (mid -6.853553 6.853553) (end -7 6.5)
       (stroke (width 0.1) (type solid)) (layer "Edge.Cuts"))
-    (fp_arc (start 6.499672 -7.000007) (mid 6.853246 -6.853571) (end 6.999672 -6.500007)
+    (fp_arc (start 6.5 -7) (mid 6.853597 -6.853597) (end 7 -6.5)
       (stroke (width 0.1) (type solid)) (layer "Edge.Cuts"))
     (fp_arc (start 7 6.5) (mid 6.853553 6.853553) (end 6.5 7)
       (stroke (width 0.1) (type solid)) (layer "Edge.Cuts"))
-    (fp_arc (start 8.40625 -7.500008) (mid 8.552696 -7.853574) (end 8.90625 -8.000008)
+    (fp_arc (start 8.563 -7.5) (mid 8.709417 -7.853583) (end 9.063 -8)
       (stroke (width 0.1) (type solid)) (layer "Edge.Cuts"))
-    (fp_arc (start 8.90625 6) (mid 8.552729 5.853536) (end 8.40625 5.5)
+    (fp_arc (start 9.063 6) (mid 8.709438 5.853562) (end 8.563 5.5)
       (stroke (width 0.1) (type solid)) (layer "Edge.Cuts"))
-    (fp_arc (start 14.90625 -8.000008) (mid 15.259774 -7.853544) (end 15.40625 -7.500008)
+    (fp_arc (start 14.813 -8) (mid 15.166539 -7.853539) (end 15.313 -7.5)
       (stroke (width 0.1) (type solid)) (layer "Edge.Cuts"))
-    (fp_arc (start 15.40625 5.5) (mid 15.259806 5.853571) (end 14.90625 6)
+    (fp_arc (start 15.313 5.5) (mid 15.166553 5.853553) (end 14.813 6)
       (stroke (width 0.1) (type solid)) (layer "Edge.Cuts"))
     (model "${ACHERONLIB}/3d_models/mx_switch.step"
@@
   (gr_line (start 185.75 82.557207) (end 185.75 116.5)
     (stroke (width 0.1) (type default)) (layer "Edge.Cuts"))
-  (gr_circle (center 210 160) (end 210 129.999999)
-    (stroke (width 0.05) (type default)) (fill none) (layer "Edge.Cuts"))
   (gr_arc (start 346.799999 80.557207) (mid 348.018231 80.971006) (end 348.732299 82.041255)
     (stroke (width 0.1) (type default)) (layer "Edge.Cuts"))
@@
   (gr_line (start 372.534289 170.882146) (end 348.732299 82.041255)
     (stroke (width 0.1) (type default)) (layer "Edge.Cuts"))
+  (gr_circle (center 210 160) (end 241 160)
+    (stroke (width 0.1) (type default)) (fill none) (layer "Edge.Cuts"))
   (gr_arc (start 372.534289 170.882146) (mid 372.334476 172.399774) (end 371.12008 173.331638)
     (stroke (width 0.1) (type default)) (layer "Edge.Cuts"))

Commit message: Updated BOM. Added new tentative plate file.
Parts:
- removed the SW27 at (166.4, 131.7)
- removed the SW27 at (161.5, 150.1)
- removed the SW51 at (322.6, 95.1)
- removed the SW51 at (341.7, 92.5)
- removed SWr: CPG151101S11, Honeydew:MX200
- added H12: M2, MountingHole:MountingHole_2.2mm_M2, F.Cu at (187.0, 222.0)
- added SW27: CPG151101S11, Honeydew:MX100, B.Cu at (166.4, 131.7)
- added SW28: CPG151101S11, Honeydew:MX100, B.Cu at (161.5, 150.1)
- added SW51: CPG151101S11, Honeydew:MX100, B.Cu at (322.6, 95.1)
- added SW56: CPG151101S11, Honeydew:MX100, B.Cu at (341.7, 92.5)
- added SW64: CPG151101S11, Honeydew:MX200, B.Cu at (210.0, 222.1)
- H4, H5, H6, H7: footprint Honeydew:MountingHole_3.2mm_M3_Pad -> MountingHole:MountingHole_3.2mm_M3; moved to B.Cu
- H8, H9: footprint Honeydew:MountingHole_3.2mm_M3_Pad -> MountingHole:MountingHole_3.2mm_M3
- moved H5 8.35 mm to (183.9, 84.6), turned to 180 degrees
- moved H4 8.35 mm to (236.0, 84.6), turned to 180 degrees
- moved H9 2.80 mm to (171.0, 215.0)
- moved H8 2.69 mm to (249.0, 215.0)
- turned H6 to 180 degrees
- turned H7 to 180 degrees
Other:
- outline, holes or cut-outs redrawn
- board text added: "SW50"
