File: PCB/Plate.kicad_pcb (KiCad board)
At the start: 2 copper layers, 325.2 x 151 mm, 71 parts, among them SW1 CPG151101S11, SW10 CPG151101S11, SW11 CPG151101S11, SW12 CPG151101S11, SW13 CPG151101S11, SW14 CPG151101S11, SW15 CPG151101S11, SW16 CPG151101S11, SW17 CPG151101S11, SW18 CPG151101S11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

Commit message: Update in progress (will be squashed)
Other:
- outline, holes or cut-outs redrawn
- board text removed: "SW50"
