File: PCB/Honeydew.kicad_sch (KiCad schematic)
At the start: 12 parts

Commit message: Added thumb wheel encoder in 2u slot.
Parts:
- added H2: M2, MountingHole:MountingHole_2.2mm_M2_Pad, symbol Mechanical:MountingHole
Other:
- sheet MCU ports: added ROTC; removed none
- sheet Matrix ports: added ROTC; removed none
- moved on the sheet: A1, H1, H2, H3

Commit message: Updated BOM. Added new tentative plate file.
Parts:
- A1: now left out of the parts list
Changed lines of the file:
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@@
   )
   (symbol (lib_id "Mechanical:Fiducial") (at 118.11 20.32 0) (unit 1)
-    (in_bom yes) (on_board yes) (dnp no)
+    (in_bom no) (on_board yes) (dnp no)
     (property "Reference" "A1" (at 120.65 19.1516 0)
       (effects (font (size 1.27 1.27)) (justify left))

Commit message: Initial V2.1 update.
Other:
- sheet MCU ports: added OLED_~{RST}; removed none
- sheet SPI ports: added OLED_~{RST}; removed none
- moved on the sheet: H1, H2
Changed lines of the file:
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@@
   (title_block
     (title "Honeydew unified split ergonomic keyboard")
-    (date "2023-04-08")
-    (rev "V2.0")
+    (date "2023-06-27")
+    (rev "V2.1")
     (company "Created by Ariamelon (https://github.com/Ariamelon/Honeydew/)")
     (comment 1 "All capacitors 50V unless otherwise specified.")
@@
     (stroke (width 0) (type default))
   )
-  (wire (pts (xy 111.76 45.72) (xy 114.3 45.72))
+  (wire (pts (xy 111.76 50.8) (xy 114.3 50.8))
     (stroke (width 0) (type default))
   )
@@
     (stroke (width 0) (type default))
   )
-  (wire (pts (xy 40.64 78.74) (xy 43.18 78.74))
+  (wire (pts (xy 40.64 81.28) (xy 43.18 81.28))
     (stroke (width 0) (type default))
   )
@@
     (stroke (width 0) (type default))
   )
-  (wire (pts (xy 111.76 45.72) (xy 111.76 48.26))
+  (wire (pts (xy 111.76 50.8) (xy 111.76 53.34))
     (stroke (width 0) (type default))
   )
@@
     (stroke (width 0) (type default))
   )
+  (wire (pts (xy 86.36 81.28) (xy 78.74 81.28))
+    (stroke (width 0) (type default))
+  )
   (symbol (lib_id "Mechanical:Fiducial") (at 118.11 20.32 0) (unit 1)
     (in_bom no) (on_board yes) (dnp no)
@@
     )
   )
-  (symbol (lib_id "Mechanical:MountingHole") (at 118.11 50.8 0) (mirror y) (unit 1)
-    (in_bom no) (on_board yes) (dnp no)
-    (property "Reference" "H2" (at 120.65 49.53 0)
-      (effects (font (size 1.27 1.27)) (justify right))
-    )
-    (property "Value" "M3" (at 120.65 52.07 0)
-      (effects (font (size 1.27 1.27)) (justify right))
-    )
-    (property "Footprint" "Honeydew:MountingHole_3.2mm_M3_Pad" (at 118.11 50.8 0)
-      (effects (font (size 1.27 1.27)) hide)
-    )
-    (property "Datasheet" "" (at 118.11 50.8 0)
-      (effects (font (size 1.27 1.27)) hide)
-    )
-    (instances
-      (project "Casaba"
-        (path "/24378b90-16c2-4770-828b-ef30a4dde4ac"
-          (reference "H2") (unit 1)
-        )
-      )
-      (project "Honeydew"
-        (path "/534caec7-cf60-4f90-b1ed-42c9d445ef0f"
-          (reference "H5") (unit 1)
+  (symbol (lib_id "Mechanical:MountingHole") (at 118.11 45.72 0) (mirror y) (unit 1)
+    (in_bom no) (on_board yes) (dnp no)
+    (property "Reference" "H2" (at 120.65 44.45 0)
+      (effects (font (size 1.27 1.27)) (justify right))
+    )
+    (property "Value" "M3" (at 120.65 46.99 0)
+      (effects (font (size 1.27 1.27)) (justify right))
+    )
+    (property "Footprint" "Honeydew:MountingHole_3.2mm_M3_Pad" (at 118.11 45.72 0)
+      (effects (font (size 1.27 1.27)) hide)
+    )
+    (property "Datasheet" "" (at 118.11 45.72 0)
+      (effects (font (size 1.27 1.27)) hide)
+    )
+    (instances
+      (project "Casaba"
+        (path "/24378b90-16c2-4770-828b-ef30a4dde4ac"
+          (reference "H2") (unit 1)
+        )
+      )
+      (project "Honeydew"
+        (path "/534caec7-cf60-4f90-b1ed-42c9d445ef0f"
+          (reference "H4") (unit 1)
         )
       )
@@
     )
   )
-  (symbol (lib_id "Mechanical:MountingHole_Pad") (at 116.84 45.72 270) (mirror x) (unit 1)
-    (in_bom no) (on_board yes) (dnp no)
-    (property "Reference" "H1" (at 120.65 44.45 90)
-      (effects (font (size 1.27 1.27)) (justify left))
-    )
-    (property "Value" "M3" (at 120.65 46.99 90)
-      (effects (font (size 1.27 1.27)) (justify left))
-    )
-    (property "Footprint" "Honeydew:MountingHole_3.2mm_M3_Pad" (at 116.84 45.72 0)
-      (effects (font (size 1.27 1.27)) hide)
-    )
-    (property "Datasheet" "" (at 116.84 45.72 0)
+  (symbol (lib_id "Mechanical:MountingHole_Pad") (at 116.84 50.8 270) (mirror x) (unit 1)
+    (in_bom no) (on_board yes) (dnp no)
+    (property "Reference" "H1" (at 120.65 49.53 90)
+      (effects (font (size 1.27 1.27)) (justify left))
+    )
+    (property "Value" "M3" (at 120.65 52.07 90)
+      (effects (font (size 1.27 1.27)) (justify left))
+    )
+    (property "Footprint" "Honeydew:MountingHole_3.2mm_M3_Pad" (at 116.84 50.8 0)
+      (effects (font (size 1.27 1.27)) hide)
+    )
+    (property "Datasheet" "" (at 116.84 50.8 0)
       (effects (font (size 1.27 1.27)) hide)
     )
@@
         )
         (path "/534caec7-cf60-4f90-b1ed-42c9d445ef0f"
-          (reference "H4") (unit 1)
+          (reference "H5") (unit 1)
         )
       )
@@
     )
   )
-  (symbol (lib_id "power:GND") (at 111.76 48.26 0) (unit 1)
+  (symbol (lib_id "power:GND") (at 111.76 53.34 0) (unit 1)
     (in_bom yes) (on_board yes) (dnp no)
-    (property "Reference" "#PWR013" (at 111.76 54.61 0)
-      (effects (font (size 1.27 1.27)) hide)
-    )
-    (property "Value" "GND" (at 111.76 52.07 0)
-      (effects (font (size 1.27 1.27)) hide)
-    )
-    (property "Footprint" "" (at 111.76 48.26 0)
-      (effects (font (size 1.27 1.27)) hide)
-    )
-    (property "Datasheet" "" (at 111.76 48.26 0)
+    (property "Reference" "#PWR013" (at 111.76 59.69 0)
+      (effects (font (size 1.27 1.27)) hide)
+    )
+    (property "Value" "GND" (at 111.76 57.15 0)
+      (effects (font (size 1.27 1.27)) hide)
+    )
+    (property "Footprint" "" (at 111.76 53.34 0)
+      (effects (font (size 1.27 1.27)) hide)
+    )
+    (property "Datasheet" "" (at 111.76 53.34 0)
       (effects (font (size 1.27 1.27)) hide)
     )
@@
     )
   )
-  (sheet (at 86.36 58.42) (size 20.32 22.86) (fields_autoplaced)
+  (sheet (at 86.36 58.42) (size 20.32 25.4) (fields_autoplaced)
     (stroke (width 0.1524) (type solid))
     (fill (color 0 0 0 0.0000))
@@
       (effects (font (size 1.27 1.27)) (justify left bottom))
     )
-    (property "Sheetfile" "SPI.kicad_sch" (at 86.36 81.8646 0)
+    (property "Sheetfile" "SPI.kicad_sch" (at 86.36 84.4046 0)
       (effects (font (size 1.27 1.27)) (justify left top) hide)
     )
@@
       (effects (font (size 1.27 1.27)) (justify left))
     )
+    (pin "OLED_~{RST}" input (at 86.36 81.28 180)
+      (effects (font (size 1.27 1.27)) (justify left))
+    )
     (instances
       (project "Honeydew"
@@
     )
   )
-  (sheet (at 20.32 76.2) (size 20.32 5.08)
+  (sheet (at 20.32 78.74) (size 20.32 5.08)
     (stroke (width 0.1524) (type solid))
     (fill (color 0 0 0 0.0000))
-    (property "Sheetname" "RGB" (at 20.32 76.2 0)
+    (property "Sheetname" "RGB" (at 20.32 78.74 0)
       (effects (font (size 1.27 1.27)) (justify left bottom))
     )
-    (property "Sheetfile" "RGB.kicad_sch" (at 38.6846 96.52 90)
+    (property "Sheetfile" "RGB.kicad_sch" (at 38.6846 99.06 90)
       (effects (font (size 1.27 1.27)) (justify left top) hide)
     )
-    (pin "RGB" input (at 40.64 78.74 0)
+    (pin "RGB" input (at 40.64 81.28 0)
       (effects (font (size 1.27 1.27)) (justify right))
     )
@@
     )
   )
-  (sheet (at 43.18 17.78) (size 35.56 63.5)
+  (sheet (at 43.18 17.78) (size 35.56 66.04)
     (stroke (width 0.1524) (type solid))
     (fill (color 0 0 0 0.0000))
@@
       (effects (font (size 1.27 1.27)) (justify right))
     )
+    (pin "OLED_~{RST}" output (at 78.74 81.28 0)
+      (effects (font (size 1.27 1.27)) (justify right))
+    )

Commit message: Routed 13V EN pin to the MCU. Removed solder jumper.
Other:
- sheet MCU ports: added 13V_EN; removed none
- sheet PSU ports: added 13V_EN; removed none
Changed lines of the file:
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@@
+    (stroke (width 0) (type default))
+  )
+  (wire (pts (xy 40.64 66.04) (xy 43.18 66.04))
+    (stroke (width 0) (type default))
+  )
+  (wire (pts (xy 86.36 35.56) (xy 78.74 35.56))
+    (stroke (width 0) (type default))
+  )
+  (wire (pts (xy 111.76 50.8) (xy 114.3 50.8))
+    (stroke (width 0) (type default))
+  )
+  (wire (pts (xy 83.82 66.04) (xy 78.74 66.04))
+    (stroke (width 0) (type default))
+  )
+  (wire (pts (xy 40.64 81.28) (xy 43.18 81.28))
+    (stroke (width 0) (type default))
+  )
+  (wire (pts (xy 81.28 45.72) (xy 81.28 60.96))
+    (stroke (width 0) (type default))
+  )
+  (wire (pts (xy 86.36 76.2) (xy 78.74 76.2))
+    (stroke (width 0) (type default))
+  )
+  (wire (pts (xy 86.36 68.58) (xy 78.74 68.58))
+    (stroke (width 0) (type default))
+  )
+  (wire (pts (xy 86.36 66.04) (xy 83.82 66.04))
+    (stroke (width 0) (type default))
+  )
+  (wire (pts (xy 40.64 53.34) (xy 43.18 53.34))
+    (stroke (width 0) (type default))
+  )
+  (wire (pts (xy 86.36 78.74) (xy 78.74 78.74))
+    (stroke (width 0) (type default))
+  )
+  (wire (pts (xy 86.36 27.94) (xy 78.74 27.94))
+    (stroke (width 0) (type default))
+  )
+  (wire (pts (xy 86.36 38.1) (xy 78.74 38.1))
+    (stroke (width 0) (type default))
+  )
+  (wire (pts (xy 43.18 40.64) (xy 40.64 40.64))
+    (stroke (width 0) (type default))
+  )
+  (wire (pts (xy 86.36 45.72) (xy 81.28 45.72))
+    (stroke (width 0) (type default))
+  )
+  (wire (pts (xy 86.36 25.4) (xy 78.74 25.4))
+    (stroke (width 0) (type default))
+  )
+  (wire (pts (xy 43.18 20.32) (xy 40.64 20.32))
+    (stroke (width 0) (type default))
+  )
+  (wire (pts (xy 81.28 60.96) (xy 78.74 60.96))
+    (stroke (width 0) (type default))
+  )
+  (wire (pts (xy 43.18 27.94) (xy 40.64 27.94))
+    (stroke (width 0) (type default))
+  )
+  (wire (pts (xy 78.74 40.64) (xy 86.36 40.64))
+    (stroke (width 0) (type default))
+  )
+  (wire (pts (xy 86.36 50.8) (xy 78.74 50.8))
+    (stroke (width 0) (type default))
+  )
+  (wire (pts (xy 86.36 20.32) (xy 78.74 20.32))
+    (stroke (width 0) (type default))
+  )
+  (wire (pts (xy 40.64 48.26) (xy 43.18 48.26))
+    (stroke (width 0) (type default))
+  )
+  (wire (pts (xy 43.18 45.72) (xy 40.64 45.72))
+    (stroke (width 0) (type default))
+  )
+  (wire (pts (xy 40.64 22.86) (xy 43.18 22.86))
+    (stroke (width 0) (type default))
+  )
+  (wire (pts (xy 86.36 48.26) (xy 83.82 48.26))
+    (stroke (width 0) (type default))
+  )
+  (wire (pts (xy 86.36 22.86) (xy 78.74 22.86))
+    (stroke (width 0) (type default))
+  )
+  (wire (pts (xy 43.18 58.42) (xy 40.64 58.42))
+    (stroke (width 0) (type default))
+  )
+  (wire (pts (xy 40.64 68.58) (xy 43.18 68.58))
+    (stroke (width 0) (type default))
+  )
+  (wire (pts (xy 86.36 71.12) (xy 78.74 71.12))
+    (stroke (width 0) (type default))
+  )
+  (wire (pts (xy 111.76 50.8) (xy 111.76 53.34))
+    (stroke (width 0) (type default))
+  )
+  (wire (pts (xy 40.64 30.48) (xy 43.18 30.48))
     (stroke (width 0) (type default))
   )
   (wire (pts (xy 40.64 60.96) (xy 43.18 60.96))
-    (stroke (width 0) (type default))
-  )
-  (wire (pts (xy 86.36 35.56) (xy 78.74 35.56))
-    (stroke (width 0) (type default))
-  )
-  (wire (pts (xy 111.76 50.8) (xy 114.3 50.8))
-    (stroke (width 0) (type default))
-  )
-  (wire (pts (xy 83.82 66.04) (xy 78.74 66.04))
-    (stroke (width 0) (type default))
-  )
-  (wire (pts (xy 40.64 81.28) (xy 43.18 81.28))
-    (stroke (width 0) (type default))
-  )
-  (wire (pts (xy 81.28 45.72) (xy 81.28 60.96))
-    (stroke (width 0) (type default))
-  )
-  (wire (pts (xy 86.36 76.2) (xy 78.74 76.2))
-    (stroke (width 0) (type default))
-  )
-  (wire (pts (xy 86.36 68.58) (xy 78.74 68.58))
-    (stroke (width 0) (type default))
-  )
-  (wire (pts (xy 86.36 66.04) (xy 83.82 66.04))
-    (stroke (width 0) (type default))
-  )
-  (wire (pts (xy 86.36 78.74) (xy 78.74 78.74))
-    (stroke (width 0) (type default))
-  )
-  (wire (pts (xy 86.36 27.94) (xy 78.74 27.94))
-    (stroke (width 0) (type default))
-  )
-  (wire (pts (xy 86.36 38.1) (xy 78.74 38.1))
-    (stroke (width 0) (type default))
-  )
-  (wire (pts (xy 43.18 40.64) (xy 40.64 40.64))
-    (stroke (width 0) (type default))
-  )
-  (wire (pts (xy 86.36 45.72) (xy 81.28 45.72))
-    (stroke (width 0) (type default))
-  )
-  (wire (pts (xy 86.36 25.4) (xy 78.74 25.4))
-    (stroke (width 0) (type default))
-  )
-  (wire (pts (xy 43.18 20.32) (xy 40.64 20.32))
-    (stroke (width 0) (type default))
-  )
-  (wire (pts (xy 81.28 60.96) (xy 78.74 60.96))
-    (stroke (width 0) (type default))
-  )
-  (wire (pts (xy 43.18 27.94) (xy 40.64 27.94))
-    (stroke (width 0) (type default))
-  )
-  (wire (pts (xy 78.74 40.64) (xy 86.36 40.64))
-    (stroke (width 0) (type default))
-  )
-  (wire (pts (xy 86.36 50.8) (xy 78.74 50.8))
-    (stroke (width 0) (type default))
-  )
-  (wire (pts (xy 86.36 20.32) (xy 78.74 20.32))
-    (stroke (width 0) (type default))
-  )
-  (wire (pts (xy 40.64 48.26) (xy 43.18 48.26))
-    (stroke (width 0) (type default))
-  )
-  (wire (pts (xy 43.18 45.72) (xy 40.64 45.72))
-    (stroke (width 0) (type default))
-  )
-  (wire (pts (xy 40.64 22.86) (xy 43.18 22.86))
-    (stroke (width 0) (type default))
-  )
-  (wire (pts (xy 86.36 48.26) (xy 83.82 48.26))
-    (stroke (width 0) (type default))
-  )
-  (wire (pts (xy 86.36 22.86) (xy 78.74 22.86))
-    (stroke (width 0) (type default))
-  )
-  (wire (pts (xy 43.18 53.34) (xy 40.64 53.34))
-    (stroke (width 0) (type default))
-  )
-  (wire (pts (xy 40.64 63.5) (xy 43.18 63.5))
-    (stroke (width 0) (type default))
-  )
-  (wire (pts (xy 86.36 71.12) (xy 78.74 71.12))
-    (stroke (width 0) (type default))
-  )
-  (wire (pts (xy 111.76 50.8) (xy 111.76 53.34))
-    (stroke (width 0) (type default))
-  )
-  (wire (pts (xy 40.64 30.48) (xy 43.18 30.48))
-    (stroke (width 0) (type default))
-  )
-  (wire (pts (xy 40.64 55.88) (xy 43.18 55.88))
     (stroke (width 0) (type default))
   )
@@
     )
   )
-  (sheet (at 20.32 38.1) (size 20.32 27.94)
+  (sheet (at 20.32 38.1) (size 20.32 33.02)
     (stroke (width 0.1524) (type solid))
     (fill (color 0 0 0 0.0000))
@@
       (effects (font (size 1.27 1.27)) (justify left) hide)
     )
-    (pin "BOARD_VSEN" output (at 40.64 53.34 0)
-      (effects (font (size 1.27 1.27)) (justify right))
-    )
-    (pin "BOARD_ILIM_~{FLT}" output (at 40.64 60.96 0)
-      (effects (font (size 1.27 1.27)) (justify right))
-    )
-    (pin "BOARD_ISEN" output (at 40.64 55.88 0)
+    (pin "BOARD_VSEN" output (at 40.64 58.42 0)
+      (effects (font (size 1.27 1.27)) (justify right))
+    )
+    (pin "BOARD_ILIM_~{FLT}" output (at 40.64 66.04 0)
+      (effects (font (size 1.27 1.27)) (justify right))
+    )
+    (pin "BOARD_ISEN" output (at 40.64 60.96 0)
       (effects (font (size 1.27 1.27)) (justify right))
     )
@@
       (effects (font (size 1.27 1.27)) (justify right))
     )
-    (pin "RGB_ILIM_~{FLT}" output (at 40.64 63.5 0)
+    (pin "RGB_ILIM_~{FLT}" output (at 40.64 68.58 0)
+      (effects (font (size 1.27 1.27)) (justify right))
+    )
+    (pin "13V_EN" input (at 40.64 53.34 0)
       (effects (font (size 1.27 1.27)) (justify right))
     )
@@
       (effects (font (size 1.27 1.27)) (justify left))
     )
-    (pin "BOARD_ISEN" input (at 43.18 55.88 180)
-      (effects (font (size 1.27 1.27)) (justify left))
-    )
-    (pin "BOARD_VSEN" input (at 43.18 53.34 180)
-      (effects (font (size 1.27 1.27)) (justify left))
-    )
-    (pin "BOARD_ILIM_~{FLT}" input (at 43.18 60.96 180)
+    (pin "BOARD_ISEN" input (at 43.18 60.96 180)
+      (effects (font (size 1.27 1.27)) (justify left))
+    )
+    (pin "BOARD_VSEN" input (at 43.18 58.42 180)
+      (effects (font (size 1.27 1.27)) (justify left))
+    )
+    (pin "BOARD_ILIM_~{FLT}" input (at 43.18 66.04 180)
       (effects (font (size 1.27 1.27)) (justify left))
     )
@@
       (effects (font (size 1.27 1.27)) (justify left))
     )
-    (pin "RGB_ILIM_~{FLT}" input (at 43.18 63.5 180)
+    (pin "RGB_ILIM_~{FLT}" input (at 43.18 68.58 180)
       (effects (font (size 1.27 1.27)) (justify left))
     )
@@
       (effects (font (size 1.27 1.27)) (justify right))
     )
-    (instances
+    (pin "13V_EN" output (at 43.18 53.34 180)
+      (effects (font (size 1.27 1.27)) (justify left))
+    )
+    (instances

Commit message: In progress update
Parts:
- H1: symbol Mechanical:MountingHole_Pad -> Mechanical:MountingHole; now in the parts list
Connections:
- removed net GND: H1.1
Other:
- sheet MCU ports: added TB_~{RST}; removed none
- sheet SPI ports: added TB_~{RST}; removed ~{RST}
- moved on the sheet: A1, H1, H2, H3
