File: PCB/Honeydew.kicad_sch (KiCad schematic)
At the start: 13 parts

Commit message: 14/07/2023 update
Replaced 1N4148 switch diodes with BAV70. Replaced switch footprints with combination MX/Choc hotswap footprints. Replaced flash IC with much smaller version. Removed buttons and USB-C port and replaced it with an FFC connector for [Galia](https://github.com/Ariamelon/Galia) (a USB-C daughterboard designed specifically for the Honeydew). Added case STEP file and renders.
Parts:
- added H2 (x3): M2, MountingHole:MountingHole_2.2mm_M2_Pad, symbol Mechanical:MountingHole
- H1: now left out of the parts list
Other:
- sheet MCU ports: added BOOTSEL; removed none
- sheet USB ports: added BOOTSEL, ~{RST}; removed none
Changed lines of the file:
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@@
   (title_block
     (title "Honeydew unified split ergonomic keyboard")
-    (date "2023-06-27")
-    (rev "V2.1")
+    (date "2023-07-14")
+    (rev "V3.0")
     (company "Created by Ariamelon (https://github.com/Ariamelon/Honeydew/)")
     (comment 1 "All capacitors 50V unless otherwise specified.")
@@
     (stroke (width 0) (type default))
   )
+  (wire (pts (xy 43.18 30.48) (xy 40.64 30.48))
+    (stroke (width 0) (type default))
+  )
   (wire (pts (xy 86.36 45.72) (xy 81.28 45.72))
     (stroke (width 0) (type default))
   )
+  (wire (pts (xy 40.64 33.02) (xy 43.18 33.02))
+    (stroke (width 0) (type default))
+  )
   (wire (pts (xy 86.36 25.4) (xy 78.74 25.4))
     (stroke (width 0) (type default))
@@
     (stroke (width 0) (type default))
   )
+  (wire (pts (xy 40.64 22.86) (xy 43.18 22.86))
+    (stroke (width 0) (type default))
+  )
   (wire (pts (xy 43.18 25.4) (xy 40.64 25.4))
     (stroke (width 0) (type default))
@@
     (stroke (width 0) (type default))
   )
-  (wire (pts (xy 40.64 22.86) (xy 43.18 22.86))
-    (stroke (width 0) (type default))
-  )
   (wire (pts (xy 86.36 48.26) (xy 83.82 48.26))
     (stroke (width 0) (type default))
@@
   )
   (symbol (lib_id "Mechanical:MountingHole") (at 116.84 50.8 270) (mirror x) (unit 1)
-    (in_bom yes) (on_board yes) (dnp no) (fields_autoplaced)
+    (in_bom no) (on_board yes) (dnp no) (fields_autoplaced)
     (property "Reference" "H1" (at 119.38 49.53 90)
       (effects (font (size 1.27 1.27)) (justify left))
@@
     )
   )
+  (symbol (lib_id "Mechanical:MountingHole") (at 129.54 55.88 0) (mirror y) (unit 1)
+    (in_bom no) (on_board yes) (dnp no)
+    (property "Reference" "H2" (at 132.08 54.61 0)
+      (effects (font (size 1.27 1.27)) (justify right))
+    )
+    (property "Value" "M2" (at 132.08 57.15 0)
+      (effects (font (size 1.27 1.27)) (justify right))
+    )
+    (property "Footprint" "MountingHole:MountingHole_2.2mm_M2_Pad" (at 129.54 55.88 0)
+      (effects (font (size 1.27 1.27)) hide)
+    )
+    (property "Datasheet" "" (at 129.54 55.88 0)
+      (effects (font (size 1.27 1.27)) hide)
+    )
+    (instances
+      (project "Casaba"
+        (path "/24378b90-16c2-4770-828b-ef30a4dde4ac"
+          (reference "H2") (unit 1)
+        )
+      )
+      (project "Honeydew"
+        (path "/534caec7-cf60-4f90-b1ed-42c9d445ef0f"
+          (reference "H14") (unit 1)
+        )
+      )
+    )
+  )
   (symbol (lib_id "Mechanical:MountingHole") (at 116.84 55.88 0) (mirror y) (unit 1)
     (in_bom no) (on_board yes) (dnp no)
@@
     )
   )
+  (symbol (lib_id "Mechanical:MountingHole") (at 129.54 50.8 0) (mirror y) (unit 1)
+    (in_bom no) (on_board yes) (dnp no)
+    (property "Reference" "H2" (at 132.08 49.53 0)
+      (effects (font (size 1.27 1.27)) (justify right))
+    )
+    (property "Value" "M2" (at 132.08 52.07 0)
+      (effects (font (size 1.27 1.27)) (justify right))
+    )
+    (property "Footprint" "MountingHole:MountingHole_2.2mm_M2_Pad" (at 129.54 50.8 0)
+      (effects (font (size 1.27 1.27)) hide)
+    )
+    (property "Datasheet" "" (at 129.54 50.8 0)
+      (effects (font (size 1.27 1.27)) hide)
+    )
+    (instances
+      (project "Casaba"
+        (path "/24378b90-16c2-4770-828b-ef30a4dde4ac"
+          (reference "H2") (unit 1)
+        )
+      )
+      (project "Honeydew"
+        (path "/534caec7-cf60-4f90-b1ed-42c9d445ef0f"
+          (reference "H13") (unit 1)
+        )
+      )
+    )
+  )
   (symbol (lib_id "Mechanical:MountingHole") (at 116.84 71.12 0) (mirror y) (unit 1)
     (in_bom no) (on_board yes) (dnp no)
@@
         (path "/534caec7-cf60-4f90-b1ed-42c9d445ef0f"
           (reference "H11") (unit 1)
+        )
+      )
+    )
+  )
+  (symbol (lib_id "Mechanical:MountingHole") (at 129.54 60.96 0) (mirror y) (unit 1)
+    (in_bom no) (on_board yes) (dnp no)
+    (property "Reference" "H2" (at 132.08 59.69 0)
+      (effects (font (size 1.27 1.27)) (justify right))
+    )
+    (property "Value" "M2" (at 132.08 62.23 0)
+      (effects (font (size 1.27 1.27)) (justify right))
+    )
+    (property "Footprint" "MountingHole:MountingHole_2.2mm_M2_Pad" (at 129.54 60.96 0)
+      (effects (font (size 1.27 1.27)) hide)
+    )
+    (property "Datasheet" "" (at 129.54 60.96 0)
+      (effects (font (size 1.27 1.27)) hide)
+    )
+    (instances
+      (project "Casaba"
+        (path "/24378b90-16c2-4770-828b-ef30a4dde4ac"
+          (reference "H2") (unit 1)
+        )
+      )
+      (project "Honeydew"
+        (path "/534caec7-cf60-4f90-b1ed-42c9d445ef0f"
+          (reference "H15") (unit 1)
         )
       )
@@
       (effects (font (size 1.27 1.27)) (justify left top) hide)
     )
-    (pin "D-" input (at 40.64 22.86 0)
-      (effects (font (size 1.27 1.27)) (justify right))
-    )
-    (pin "D+" output (at 40.64 20.32 0)
-      (effects (font (size 1.27 1.27)) (justify right))
-    )
     (pin "TUSB_OUT1" output (at 40.64 25.4 0)
       (effects (font (size 1.27 1.27)) (justify right))
     )
     (pin "TUSB_OUT2" output (at 40.64 27.94 0)
+      (effects (font (size 1.27 1.27)) (justify right))
+    )
+    (pin "BOOTSEL" output (at 40.64 33.02 0)
+      (effects (font (size 1.27 1.27)) (justify right))
+    )
+    (pin "~{RST}" output (at 40.64 30.48 0)
+      (effects (font (size 1.27 1.27)) (justify right))
+    )
+    (pin "D-" bidirectional (at 40.64 22.86 0)
+      (effects (font (size 1.27 1.27)) (justify right))
+    )
+    (pin "D+" bidirectional (at 40.64 20.32 0)
       (effects (font (size 1.27 1.27)) (justify right))
     )
@@
       (effects (font (size 1.27 1.27)) (justify left top) hide)
     )
-    (pin "D-" output (at 43.18 22.86 180)
-      (effects (font (size 1.27 1.27)) (justify left))
-    )
-    (pin "D+" input (at 43.18 20.32 180)
-      (effects (font (size 1.27 1.27)) (justify left))
-    )
     (pin "ROW1" input (at 78.74 22.86 0)
       (effects (font (size 1.27 1.27)) (justify right))
@@
       (effects (font (size 1.27 1.27)) (justify left))
     )
-    (pin "~{RST}" output (at 43.18 30.48 180)
-      (effects (font (size 1.27 1.27)) (justify left))
-    )
     (pin "TB_~{RST}" output (at 78.74 68.58 0)
       (effects (font (size 1.27 1.27)) (justify right))
     )
-    (instances
+    (pin "D+" bidirectional (at 43.18 20.32 180)
+      (effects (font (size 1.27 1.27)) (justify left))
+    )
+    (pin "D-" bidirectional (at 43.18 22.86 180)
+      (effects (font (size 1.27 1.27)) (justify left))
+    )
+    (pin "~{RST}" input (at 43.18 30.48 180)
+      (effects (font (size 1.27 1.27)) (justify left))
+    )
+    (pin "BOOTSEL" input (at 43.18 33.02 180)
+      (effects (font (size 1.27 1.27)) (justify left))
+    )
+    (instances
