File: PCB/Plate Scroll.kicad_pcb (KiCad board)
At the start: 2 copper layers, 334.8 x 169.6 mm, 63 parts, among them SW1 CPG151101S11, SW10 CPG151101S11, SW11 CPG151101S11, SW12 CPG151101S11, SW13 CPG151101S11, SW14 CPG151101S11, SW15 CPG151101S11, SW16 CPG151101S11, SW17 CPG151101S11, SW18 CPG151101S11, SW19 CPG151101S11, SW2 CPG151101S11, SW20 CPG151101S11, SW21 CPG151101S11, SW22 CPG151101S11, SW23 CPG151101S11, SW24 CPG151101S11, SW25 CPG151101S11, SW26 CPG151101S11, SW27 CPG151101S11, SW28 CPG151101S11, SW29 CPG151101S11, SW3 CPG151101S11, SW30 CPG151101S11, SW31 CPG151101S11, SW32 CPG151101S11, SW33 CPG151101S11, SW34 CPG151101S11, SW35 CPG151101S11, SW36 CPG151101S11, SW37 CPG151101S11, SW38 CPG151101S11, SW39 CPG151101S11, SW4 CPG151101S11, SW40 CPG151101S11, SW41 CPG151101S11, SW42 CPG151101S11, SW43 CPG151101S11, SW44 CPG151101S11, SW45 CPG151101S11, SW46 CPG151101S11, SW47 CPG151101S11, SW48 CPG151101S11, SW49 CPG151101S11, SW5 CPG151101S11, SW50 CPG151101S11, SW51 CPG151101S11, SW52 CPG151101S11, SW53 CPG151101S11, SW54 CPG151101S11, SW55 CPG151101S11, SW56 CPG151101S11, SW57 CPG151101S11, SW58 CPG151101S11, SW59 CPG151101S11, SW6 CPG151101S11, SW60 CPG151101S11, SW61 CPG151101S11, SW62 CPG151101S11, SW63 CPG151101S11, SW7 CPG151101S11, SW8 CPG151101S11, SW9 CPG151101S11

Commit message: 26/07/2023 update
Sent to JLC (V3.0 release version). Slightly increased size of screw hole pads. Added two more screw holes. Added mounting holes to plate. Flipped gerbers for scrollwheel plate.
Parts:
- added REF**: MountingHole_3.2mm_M3, MountingHole:MountingHole_3.2mm_M3, F.Cu at (237.5, 83.9)
- added REF**: MountingHole_3.2mm_M3, MountingHole:MountingHole_3.2mm_M3, F.Cu at (315.9, 83.9)
- added REF**: MountingHole_3.2mm_M3, MountingHole:MountingHole_3.2mm_M3, F.Cu at (182.5, 83.9)
- added REF**: MountingHole_3.2mm_M3, MountingHole:MountingHole_3.2mm_M3, F.Cu at (171.0, 215.0)
- added REF**: MountingHole_3.2mm_M3, MountingHole:MountingHole_3.2mm_M3, F.Cu at (87.7, 180.2)
- added REF**: MountingHole_3.2mm_M3, MountingHole:MountingHole_3.2mm_M3, F.Cu at (332.3, 180.2)
- added REF**: MountingHole_3.2mm_M3, MountingHole:MountingHole_3.2mm_M3, F.Cu at (249.0, 215.0)
- added REF**: MountingHole_3.2mm_M3, MountingHole:MountingHole_3.2mm_M3, F.Cu at (104.1, 83.9)
Other:
- outline, holes or cut-outs redrawn

Commit message: 30/07/2023 update
Added VIK keyboard certification card. Added USB connector back to PCB, but left the two buttons on a separate daughterboard. Modified case to accommodate large VIK module.
Parts:
- moved REF** 2.72 mm to (237.5, 86.6)
- moved REF** 2.72 mm to (315.9, 86.6)
- moved REF** 2.72 mm to (182.5, 86.6)
- moved REF** 2.72 mm to (171.0, 217.7)
- moved REF** 2.72 mm to (87.7, 182.9)
- moved REF** 2.72 mm to (332.3, 182.9)
- moved REF** 2.72 mm to (249.0, 217.7)
- moved REF** 2.72 mm to (104.1, 86.6)
- moved SW1 2.72 mm to (78.3, 95.2)
- moved SW10 2.72 mm to (77.6, 171.4)
- moved SW11 2.72 mm to (117.0, 98.2)
- moved SW12 2.72 mm to (112.1, 116.6)
- moved SW13 2.72 mm to (107.1, 135.0)
- moved SW14 2.72 mm to (102.2, 153.4)
- moved SW15 2.72 mm to (97.3, 171.8)
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Other:
- outline, holes or cut-outs redrawn
