File: Case/Plate Scroll.kicad_pcb (KiCad board)
At the start: 2 copper layers, 334.8 x 169.6 mm, 71 parts, among them SW1 CPG151101S11, SW10 CPG151101S11, SW11 CPG151101S11, SW12 CPG151101S11, SW13 CPG151101S11, SW14 CPG151101S11, SW15 CPG151101S11, SW16 CPG151101S11, SW17 CPG151101S11, SW18 CPG151101S11, SW19 CPG151101S11, SW2 CPG151101S11, SW20 CPG151101S11, SW21 CPG151101S11, SW22 CPG151101S11, SW23 CPG151101S11, SW24 CPG151101S11, SW25 CPG151101S11, SW26 CPG151101S11, SW27 CPG151101S11, SW28 CPG151101S11, SW29 CPG151101S11, SW3 CPG151101S11, SW30 CPG151101S11, SW31 CPG151101S11, SW32 CPG151101S11, SW33 CPG151101S11, SW34 CPG151101S11, SW35 CPG151101S11, SW36 CPG151101S11, SW37 CPG151101S11, SW38 CPG151101S11, SW39 CPG151101S11, SW4 CPG151101S11, SW40 CPG151101S11, SW41 CPG151101S11, SW42 CPG151101S11, SW43 CPG151101S11, SW44 CPG151101S11, SW45 CPG151101S11, SW46 CPG151101S11, SW47 CPG151101S11, SW48 CPG151101S11, SW49 CPG151101S11, SW5 CPG151101S11, SW50 CPG151101S11, SW51 CPG151101S11, SW52 CPG151101S11, SW53 CPG151101S11, SW54 CPG151101S11, SW55 CPG151101S11, SW56 CPG151101S11, SW57 CPG151101S11, SW58 CPG151101S11, SW59 CPG151101S11, SW6 CPG151101S11, SW60 CPG151101S11, SW61 CPG151101S11, SW62 CPG151101S11, SW63 CPG151101S11, SW7 CPG151101S11, SW8 CPG151101S11, SW9 CPG151101S11

Commit message: 31/07/2023 update
Removed button daughterboard. Reduced size of case and gaskets and added locating features. Added o-ring mounting for the PCB to the bottom case. Added fittings BOM.
Other:
- board size 334.8 x 169.6 mm -> 331.9 x 166.1 mm

Commit message: 01/08/2023 update
Removed 3D files for trackpad mount and knob, moved to Kiwano repository. Increased size of center hole in plate. Increased size of center hole in plate. Added renders with trackball configurations (refer to Kiwano).
Parts:
- removed REF** (x8): MountingHole_3.2mm_M3, MountingHole:MountingHole_3.2mm_M3
Other:
- outline, holes or cut-outs redrawn

Commit message: 08/05/2023 update
Fixed switch and SK6812 MINI-E footprints to get rid of DRC errors. Fixed EC10 footprint and merged together PTS645 and D2F footprints. Fixed plate files to fit JLC 1.6mm minimum slot specification. Added fusion file for overall design.
Other:
- outline, holes or cut-outs redrawn

Commit message: 17/08/2023 update
Moved gasket mounts from plate to PCB. Changed USB C connector. Modified case to accommodate. Tweaked thumb scroll holder.
Other:
- board size 331.9 x 166.1 mm -> 329.7 x 154.7 mm

Commit message: 27/08/2023 update
Added unified library for all symbols, footprints and 3D files. Changed MCU to STM32F072RBT6. Removed OLED, voltage and current sensing, USB CC circuitry and shift registers. Changed ESD protection chip. Cleaned up routing and component placement. Changed SWD header pinout to 6-pin standard.
Other:
- outline, holes or cut-outs redrawn
